File: ShieldBluepill V2/Arquivos kicad/Shield STM32 Bluepill.kicad_pcb (KiCad board)
At the start: 2 copper layers, 99 x 90.1 mm, 76 parts, among them J1 Screw_Terminal_01x02, J10 PWM/ADC1, J11 Serial, J12 SPI_2, J13 Bluetooth ZS-040, J14 Acelerometro GY-521, J15 SD CARD, J16 Display OLED 0.96'', J17 Modulo WIFI ESP01, J2 Screw_Terminal_01x02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

Commit message: REV 0.0
Routing:
- net +3V3: track 311.6 -> 315.9 mm
- net /PA2: track 41.6 -> 41.1 mm
Other:
- board text added: "Rev. 0.0 - 04/2024"
- board text added: "https://github.com/Rdisrael/Projeto-Bluepill"
- board text removed: "Rev. 2.0 - 04/2024"
